Commit message: workaround to spawn tp flange description

File: kuka_lbr_iiwa_support/urdf/lbr_iiwa14_r820_macro.xacro (robot description, xacro)
@@ -141,12 +141,12 @@
       <visual>
         <geometry>
-          <mesh filename="package://${package_name}/meshes/lbr_iiwa14_r820/visual/link_7.dae"/>
-        </geometry>
-        <origin rpy="0.0 0.0 0.0" xyz="0.0 0.0 0.0"/>
-      </visual>
-      <collision>
-        <origin rpy="0.0 0.0 0.0" xyz="0.0 0.0 0.0"/>
-        <geometry>
-          <mesh filename="package://${package_name}/meshes/lbr_iiwa14_r820/collision/link_7.stl"/>
+          <mesh filename="package://${package_name}/meshes/lbr_iiwa14_r820/visual/link_7_tp.dae"/>
+        </geometry>
+        <origin rpy="0.0 0.0 0.0" xyz="0.0 0.0 0.0"/>
+      </visual>
+      <collision>
+        <origin rpy="0.0 0.0 0.0" xyz="0.0 0.0 0.0"/>
+        <geometry>
+          <mesh filename="package://${package_name}/meshes/lbr_iiwa14_r820/collision/link_7_tp.stl"/>
         </geometry>
       </collision>
@@ -224,5 +224,5 @@
       <parent link="${prefix}link_7"/>
       <child link="${prefix}flange"/>
-      <origin rpy="0.0 0.0 0.0" xyz="0.0 0.0 0.045"/>
+      <origin rpy="0.0 0.0 0.0" xyz="0.0 0.0 0.071"/>
     </joint>
     <!-- ROS-Industrial 'tool0' frame - all-zeros tool frame -->
@@ -231,5 +231,5 @@
       <parent link="${prefix}link_7"/>
       <child link="${prefix}tool0"/>
-      <origin rpy="0.0 0.0 0.0" xyz="0.0 0.0 0.045"/>
+      <origin rpy="0.0 0.0 0.0" xyz="0.0 0.0 0.071"/>
     </joint>
   </xacro:macro>
